File: isoUARTTranceiver.kicad_sch (KiCad schematic)
At the start: 20 parts, among them U2 TLE9015DQUXUMA1

Commit message: minor changes
Parts:
- R15: footprint (none) -> Resistor_SMD:R_0603_1608Metric
Changed lines of the file:
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@@
 			)
 		)
-		(property "Footprint" ""
+		(property "Footprint" "Resistor_SMD:R_0603_1608Metric"
 			(at 179.07 139.7 0)
 			(hide yes)
