File: CANTranceiver.kicad_sch (KiCad schematic)
At the start: 9 parts, among them U3 IC TRANSCEIVER 1/1 8SO

Commit message: initial component placement
Parts:
- renumbered C2 to C18, C9 to C19, C13 to C20, C11 to C21, D4 to D2, D5 to D3, R10 to R20, R11 to R21
Changed lines of the file:
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@@
 		(dnp no)
 		(fields_autoplaced yes)
-		(property "Reference" "#PWR051"
+		(property "Reference" "#PWR044"
 			(at 128.27 147.32 0)
 			(hide yes)
@@
 			(project "bms-main"
 				(path "/d7e1c873-142c-4805-8303-47f5b9830fe8/3499863e-1965-40fb-acb8-8c0f2bec52b8"
-					(reference "#PWR051")
+					(reference "#PWR044")
 					(unit 1)
 				)
@@
 		(in_pos_files yes)
 		(dnp no)
-		(property "Reference" "C2"
+		(property "Reference" "C18"
 			(at 76.2 56.896 0)
 			(show_name no)
@@
 			(project "bms-main"
 				(path "/d7e1c873-142c-4805-8303-47f5b9830fe8/3499863e-1965-40fb-acb8-8c0f2bec52b8"
-					(reference "C2")
+					(reference "C18")
 					(unit 1)
 				)
@@
 		(dnp no)
 		(fields_autoplaced yes)
-		(property "Reference" "C11"
+		(property "Reference" "C21"
 			(at 198.12 67.3162 0)
 			(show_name no)
@@
 			(project "bms-main"
 				(path "/d7e1c873-142c-4805-8303-47f5b9830fe8/3499863e-1965-40fb-acb8-8c0f2bec52b8"
-					(reference "C11")
+					(reference "C21")
 					(unit 1)
 				)
@@
 		(in_pos_files yes)
 		(dnp no)
-		(property "Reference" "D4"
+		(property "Reference" "D2"
 			(at 120.142 99.06 90)
 			(show_name no)
@@
 			(project "bms-main"
 				(path "/d7e1c873-142c-4805-8303-47f5b9830fe8/3499863e-1965-40fb-acb8-8c0f2bec52b8"
-					(reference "D4")
+					(reference "D2")
 					(unit 1)
 				)
@@
 		(in_pos_files yes)
 		(dnp no)
-		(property "Reference" "R11"
+		(property "Reference" "R21"
 			(at 136.906 114.3 0)
 			(show_name no)
@@
 			(project "bms-main"
 				(path "/d7e1c873-142c-4805-8303-47f5b9830fe8/3499863e-1965-40fb-acb8-8c0f2bec52b8"
-					(reference "R11")
+					(reference "R21")
 					(unit 1)
 				)
@@
 		(dnp no)
 		(fields_autoplaced yes)
-		(property "Reference" "#PWR017"
+		(property "Reference" "#PWR041"
 			(at 87.63 73.66 0)
 			(hide yes)
@@
 			(project "bms-main"
 				(path "/d7e1c873-142c-4805-8303-47f5b9830fe8/3499863e-1965-40fb-acb8-8c0f2bec52b8"
-					(reference "#PWR017")
+					(reference "#PWR041")
 					(unit 1)
 				)
@@
 		(dnp no)
 		(fields_autoplaced yes)
-		(property "Reference" "C13"
+		(property "Reference" "C20"
 			(at 157.48 111.7662 0)
 			(show_name no)
@@
 			(project "bms-main"
 				(path "/d7e1c873-142c-4805-8303-47f5b9830fe8/3499863e-1965-40fb-acb8-8c0f2bec52b8"
-					(reference "C13")
+					(reference "C20")
 					(unit 1)
 				)
@@
 		(dnp no)
 		(fields_autoplaced yes)
-		(property "Reference" "#PWR026"
+		(property "Reference" "#PWR047"
 			(at 195.58 80.01 0)
 			(hide yes)
@@
 			(project "bms-main"
 				(path "/d7e1c873-142c-4805-8303-47f5b9830fe8/3499863e-1965-40fb-acb8-8c0f2bec52b8"
-					(reference "#PWR026")
+					(reference "#PWR047")
 					(unit 1)
 				)
@@
 		(dnp no)
 		(fields_autoplaced yes)
-		(property "Reference" "#PWR027"
+		(property "Reference" "#PWR046"
 			(at 195.58 64.77 0)
 			(hide yes)
@@
 			(project "bms-main"
 				(path "/d7e1c873-142c-4805-8303-47f5b9830fe8/3499863e-1965-40fb-acb8-8c0f2bec52b8"
-					(reference "#PWR027")
+					(reference "#PWR046")
 					(unit 1)
 				)
@@
 		(dnp no)
 		(fields_autoplaced yes)
-		(property "Reference" "#PWR028"
+		(property "Reference" "#PWR040"
 			(at 80.01 73.66 0)
 			(hide yes)
@@
 			(project "bms-main"
 				(path "/d7e1c873-142c-4805-8303-47f5b9830fe8/3499863e-1965-40fb-acb8-8c0f2bec52b8"
-					(reference "#PWR028")
+					(reference "#PWR040")
 					(unit 1)
 				)
@@
 		(dnp no)
 		(fields_autoplaced yes)
-		(property "Reference" "#PWR029"
+		(property "Reference" "#PWR045"
 			(at 154.94 123.19 0)
 			(hide yes)
@@
 			(project "bms-main"
 				(path "/d7e1c873-142c-4805-8303-47f5b9830fe8/3499863e-1965-40fb-acb8-8c0f2bec52b8"
-					(reference "#PWR029")
+					(reference "#PWR045")
 					(unit 1)
 				)
@@
 		(in_pos_files yes)
 		(dnp no)
-		(property "Reference" "#PWR018"
+		(property "Reference" "#PWR039"
 			(at 80.01 57.15 0)
 			(hide yes)
@@
 			(project "bms-main"
 				(path "/d7e1c873-142c-4805-8303-47f5b9830fe8/3499863e-1965-40fb-acb8-8c0f2bec52b8"
-					(reference "#PWR018")
+					(reference "#PWR039")
 					(unit 1)
 				)
@@
 		(dnp no)
 		(fields_autoplaced yes)
-		(property "Reference" "R10"
+		(property "Reference" "R20"
 			(at 146.05 101.5999 0)
 			(show_name no)
@@
 			(project "bms-main"
 				(path "/d7e1c873-142c-4805-8303-47f5b9830fe8/3499863e-1965-40fb-acb8-8c0f2bec52b8"
-					(reference "R10")
+					(reference "R20")
 					(unit 1)
 				)
@@
 		(dnp no)
 		(fields_autoplaced yes)
-		(property "Reference" "#PWR016"
+		(property "Reference" "#PWR042"
 			(at 125.73 73.66 0)
 			(hide yes)
@@
 			(project "bms-main"
 				(path "/d7e1c873-142c-4805-8303-47f5b9830fe8/3499863e-1965-40fb-acb8-8c0f2bec52b8"
-					(reference "#PWR016")
+					(reference "#PWR042")
 					(unit 1)
 				)
@@
 		(dnp no)
 		(fields_autoplaced yes)
-		(property "Reference" "D5"
+		(property "Reference" "D3"
 			(at 130.81 133.3499 90)
 			(show_name no)
@@
 			(project "bms-main"
 				(path "/d7e1c873-142c-4805-8303-47f5b9830fe8/3499863e-1965-40fb-acb8-8c0f2bec52b8"
-					(reference "D5")
+					(reference "D3")
 					(unit 1)
 				)
@@
 		(dnp no)
 		(fields_autoplaced yes)
-		(property "Reference" "C9"
+		(property "Reference" "C19"
 			(at 90.17 59.6962 0)
 			(show_name no)
@@
 			(project "bms-main"
 				(path "/d7e1c873-142c-4805-8303-47f5b9830fe8/3499863e-1965-40fb-acb8-8c0f2bec52b8"
-					(reference "C9")
-					(unit 1)
-				)
+					(reference "C19")
+					(unit 1)
+				)

Commit message: 2 layer
Connections:
- net CANH_P renamed CAN_P
- net CANL_N renamed CAN_N
Changed lines of the file:
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@@
 		)
 	)
-	(hierarchical_label "CANH_P"
+	(hierarchical_label "CAN_P"
 		(shape input)
 		(at 121.92 93.98 180)
@@
 		)
 	)
-	(hierarchical_label "CANL_N"
+	(hierarchical_label "CAN_N"
 		(shape input)
 		(at 177.8 60.96 0)
@@
 		)
 	)
-	(hierarchical_label "CANH_P"
+	(hierarchical_label "CAN_P"
 		(shape input)
 		(at 177.8 58.42 0)
@@
 		)
 	)
-	(hierarchical_label "CANL_N"
+	(hierarchical_label "CAN_N"
 		(shape input)
 		(at 121.92 127 180)

Commit message: layout review
Changed lines of the file:
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@@
+	)
+	(junction
+		(at 127 93.98)
+		(diameter 0)
+		(color 0 0 0 0)
 	)
 	(junction
@@
 	)
 	(junction
-		(at 127 93.98)
-		(diameter 0)
-		(color 0 0 0 0)
-	)
-	(junction
 		(at 87.63 55.88)
 		(diameter 0)
@@
 	(wire
 		(pts
-			(xy 121.92 93.98) (xy 127 93.98)
+			(xy 120.65 93.98) (xy 127 93.98)
 		)
 		(stroke
@@
 	(hierarchical_label "CAN_P"
 		(shape input)
-		(at 121.92 93.98 180)
+		(at 120.65 93.98 180)
 		(effects
 			(font
