File: CurrentSense.kicad_sch (KiCad schematic)
At the start: 5 parts, among them J3 XT60PW-M, J8 XT60PW-M, U4 INA181A3IDBVR

Commit message: initial component placement
Parts:
- renumbered C28 to C22, J3 to J6, J8 to J7, R12 to R22
Changed lines of the file:
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@@
 		(dnp no)
 		(fields_autoplaced yes)
-		(property "Reference" "#PWR035"
+		(property "Reference" "#PWR054"
 			(at 193.04 124.46 0)
 			(hide yes)
@@
 			(project "bms-main"
 				(path "/d7e1c873-142c-4805-8303-47f5b9830fe8/fcf0b0b9-3f68-46bd-a825-62168094e731"
-					(reference "#PWR035")
+					(reference "#PWR054")
 					(unit 1)
 				)
@@
 		(dnp no)
 		(fields_autoplaced yes)
-		(property "Reference" "#PWR034"
+		(property "Reference" "#PWR052"
 			(at 157.48 124.46 0)
 			(hide yes)
@@
 			(project "bms-main"
 				(path "/d7e1c873-142c-4805-8303-47f5b9830fe8/fcf0b0b9-3f68-46bd-a825-62168094e731"
-					(reference "#PWR034")
+					(reference "#PWR052")
 					(unit 1)
 				)
@@
 		(dnp no)
 		(fields_autoplaced yes)
-		(property "Reference" "J3"
+		(property "Reference" "J6"
 			(at 100.33 119.3799 0)
 			(show_name no)
@@
 			(project "bms-main"
 				(path "/d7e1c873-142c-4805-8303-47f5b9830fe8/fcf0b0b9-3f68-46bd-a825-62168094e731"
-					(reference "J3")
+					(reference "J6")
 					(unit 1)
 				)
@@
 		(dnp no)
 		(fields_autoplaced yes)
-		(property "Reference" "#PWR033"
+		(property "Reference" "#PWR053"
 			(at 161.29 88.9 0)
 			(hide yes)
@@
 			(project "bms-main"
 				(path "/d7e1c873-142c-4805-8303-47f5b9830fe8/fcf0b0b9-3f68-46bd-a825-62168094e731"
-					(reference "#PWR033")
+					(reference "#PWR053")
 					(unit 1)
 				)
@@
 		(dnp no)
 		(fields_autoplaced yes)
-		(property "Reference" "C28"
+		(property "Reference" "C22"
 			(at 163.83 76.2062 0)
 			(show_name no)
@@
 			(project "bms-main"
 				(path "/d7e1c873-142c-4805-8303-47f5b9830fe8/fcf0b0b9-3f68-46bd-a825-62168094e731"
-					(reference "C28")
+					(reference "C22")
 					(unit 1)
 				)
@@
 		(dnp no)
 		(fields_autoplaced yes)
-		(property "Reference" "#PWR032"
+		(property "Reference" "#PWR051"
 			(at 154.94 73.66 0)
 			(hide yes)
@@
 			(project "bms-main"
 				(path "/d7e1c873-142c-4805-8303-47f5b9830fe8/fcf0b0b9-3f68-46bd-a825-62168094e731"
-					(reference "#PWR032")
+					(reference "#PWR051")
 					(unit 1)
 				)
@@
 		(in_pos_files yes)
 		(dnp no)
-		(property "Reference" "#PWR031"
+		(property "Reference" "#PWR050"
 			(at 121.92 138.43 0)
 			(hide yes)
@@
 			(project "bms-main"
 				(path "/d7e1c873-142c-4805-8303-47f5b9830fe8/fcf0b0b9-3f68-46bd-a825-62168094e731"
-					(reference "#PWR031")
+					(reference "#PWR050")
 					(unit 1)
 				)
@@
 		(dnp no)
 		(fields_autoplaced yes)
-		(property "Reference" "R12"
+		(property "Reference" "R22"
 			(at 134.62 105.4099 0)
 			(show_name no)
@@
 			(project "bms-main"
 				(path "/d7e1c873-142c-4805-8303-47f5b9830fe8/fcf0b0b9-3f68-46bd-a825-62168094e731"
-					(reference "R12")
+					(reference "R22")
 					(unit 1)
 				)
@@
 		(dnp no)
 		(fields_autoplaced yes)
-		(property "Reference" "J8"
+		(property "Reference" "J7"
 			(at 102.87 93.9799 0)
 			(show_name no)
@@
 			(project "bms-main"
 				(path "/d7e1c873-142c-4805-8303-47f5b9830fe8/fcf0b0b9-3f68-46bd-a825-62168094e731"
-					(reference "J8")
+					(reference "J7")
 					(unit 1)
 				)
@@
 		(dnp no)
 		(fields_autoplaced yes)
-		(property "Reference" "#PWR042"
+		(property "Reference" "#PWR048"
 			(at 121.92 93.98 0)
 			(hide yes)
@@
 			(project "bms-main"
 				(path "/d7e1c873-142c-4805-8303-47f5b9830fe8/fcf0b0b9-3f68-46bd-a825-62168094e731"
-					(reference "#PWR042")
+					(reference "#PWR048")
 					(unit 1)
 				)

Commit message: switched to 4 layer and added traces
Connections:
- net BAT_GND is gone; now on net GND: J6.1 (P), J6.2 (N), J6.SH1 (SHIELD), J6.SH2 (SHIELD), J7.SH1 (SHIELD), J7.SH2 (SHIELD), R22.2, U4.4 (IN-)
Changed lines of the file:
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@@
 	(wire
 		(pts
-			(xy 121.92 99.06) (xy 121.92 101.6)
+			(xy 121.92 99.06) (xy 121.92 102.87)
 		)
 		(stroke
@@
 	(symbol
 		(lib_id "power:GNDREF")
-		(at 121.92 101.6 0)
+		(at 121.92 102.87 0)
 		(mirror y)
 		(unit 1)
@@
 		(dnp no)
 		(property "Reference" "#PWR049"
-			(at 121.92 107.95 0)
-			(hide yes)
-			(show_name no)
-			(do_not_autoplace no)
-			(effects
-				(font
-					(size 1.27 1.27)
-				)
-			)
-		)
-		(property "Value" "BAT_GND"
-			(at 110.998 103.378 0)
+			(at 121.92 109.22 0)
+			(hide yes)
+			(show_name no)
+			(do_not_autoplace no)
+			(effects
+				(font
+					(size 1.27 1.27)
+				)
+			)
+		)
+		(property "Value" "GND"
+			(at 124.46 104.648 0)
 			(show_name no)
 			(do_not_autoplace no)
@@
 		)
 		(property "Footprint" ""
-			(at 121.92 101.6 0)
+			(at 121.92 102.87 0)
 			(hide yes)
 			(show_name no)
@@
 		)
 		(property "Datasheet" ""
-			(at 121.92 101.6 0)
+			(at 121.92 102.87 0)
 			(hide yes)
 			(show_name no)
@@
 		)
 		(property "Description" "Power symbol creates a global label with name \"GNDREF\" , reference supply ground"
-			(at 121.92 101.6 0)
+			(at 121.92 102.87 0)
 			(hide yes)
 			(show_name no)
@@
 			)
 		)
-		(property "Value" "BAT_GND"
-			(at 118.364 136.906 0)
-			(show_name no)
-			(do_not_autoplace no)
+		(property "Value" "GND"
+			(at 119.888 137.16 0)
+			(show_name no)
+			(do_not_autoplace no)
