File: bms-main.kicad_sch (KiCad schematic)
At the start: 4 parts, among them J1 CONN HEADER VERT 2POS 1.5MM, J4 CONN HEADER VERT 2POS 1.5MM, J5 CONN HEADER VERT 2POS 1.5MM, J6 CONN HEADER VERT 4POS 2.5MM

Commit message: initial component placement
Parts:
- renumbered J5 to J2, J4 to J3, J6 to J4
Changed lines of the file:
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@@
 		(dnp no)
 		(fields_autoplaced yes)
-		(property "Reference" "#PWR025"
+		(property "Reference" "#PWR05"
 			(at 212.09 72.39 0)
 			(hide yes)
@@
 			(project "bms-main"
 				(path "/d7e1c873-142c-4805-8303-47f5b9830fe8"
-					(reference "#PWR025")
+					(reference "#PWR05")
 					(unit 1)
 				)
@@
 		(dnp no)
 		(fields_autoplaced yes)
-		(property "Reference" "J4"
+		(property "Reference" "J3"
 			(at 67.31 168.9099 0)
 			(show_name no)
@@
 			(project "bms-main"
 				(path "/d7e1c873-142c-4805-8303-47f5b9830fe8"
-					(reference "J4")
+					(reference "J3")
 					(unit 1)
 				)
@@
 		(dnp no)
 		(fields_autoplaced yes)
-		(property "Reference" "#PWR022"
+		(property "Reference" "#PWR03"
 			(at 50.8 171.45 0)
 			(hide yes)
@@
 			(project "bms-main"
 				(path "/d7e1c873-142c-4805-8303-47f5b9830fe8"
-					(reference "#PWR022")
+					(reference "#PWR03")
 					(unit 1)
 				)
@@
 		(dnp no)
 		(fields_autoplaced yes)
-		(property "Reference" "#PWR024"
+		(property "Reference" "#PWR02"
 			(at 50.8 157.48 0)
 			(hide yes)
@@
 			(project "bms-main"
 				(path "/d7e1c873-142c-4805-8303-47f5b9830fe8"
-					(reference "#PWR024")
+					(reference "#PWR02")
 					(unit 1)
 				)
@@
 		(dnp no)
 		(fields_autoplaced yes)
-		(property "Reference" "#PWR023"
+		(property "Reference" "#PWR01"
 			(at 50.8 148.59 0)
 			(hide yes)
@@
 			(project "bms-main"
 				(path "/d7e1c873-142c-4805-8303-47f5b9830fe8"
-					(reference "#PWR023")
+					(reference "#PWR01")
 					(unit 1)
 				)
@@
 		(dnp no)
 		(fields_autoplaced yes)
-		(property "Reference" "J5"
+		(property "Reference" "J2"
 			(at 67.31 146.0499 0)
 			(show_name no)
@@
 			(project "bms-main"
 				(path "/d7e1c873-142c-4805-8303-47f5b9830fe8"
-					(reference "J5")
+					(reference "J2")
 					(unit 1)
 				)
@@
 		(dnp no)
 		(fields_autoplaced yes)
-		(property "Reference" "#PWR021"
+		(property "Reference" "#PWR04"
 			(at 50.8 180.34 0)
 			(hide yes)
@@
 			(project "bms-main"
 				(path "/d7e1c873-142c-4805-8303-47f5b9830fe8"
-					(reference "#PWR021")
+					(reference "#PWR04")
 					(unit 1)
 				)
@@
 		(dnp no)
 		(fields_autoplaced yes)
-		(property "Reference" "J6"
+		(property "Reference" "J4"
 			(at 228.6 58.4199 0)
 			(show_name no)
@@
 			(project "bms-main"
 				(path "/d7e1c873-142c-4805-8303-47f5b9830fe8"
-					(reference "J6")
-					(unit 1)
-				)
+					(reference "J4")
+					(unit 1)
+				)

Commit message: 2 layer
Connections:
- net CANTranceiver/CANH_P renamed CANTranceiver/CAN_P
- net CANTranceiver/CANL_N renamed CANTranceiver/CAN_N
Other:
- sheet CANTranceiver ports: added CAN_N, CAN_P; removed CANH_P, CANL_N
Changed lines of the file:
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@@
 			)
 		)
-		(pin "CANL_N" input
+		(pin "CAN_N" input
 			(at 194.31 60.96 0)
 			(effects
@@
 			)
 		)
-		(pin "CANH_P" input
+		(pin "CAN_P" input
 			(at 194.31 58.42 0)
 			(effects

Commit message: layout review
Connections:
- net isoUARTTranceiver/IFH_H renamed isoUARTTranceiver/IFH_P
- net isoUARTTranceiver/IFH_L renamed isoUARTTranceiver/IFH_N
Other:
- sheet isoUARTTranceiver ports: added IFH_N, IFH_P; removed IFH_H, IFH_L
Changed lines of the file:
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@@
 			)
 		)
-		(pin "IFH_L" input
+		(pin "IFH_N" input
 			(at 66.04 57.15 180)
 			(effects
@@
 			)
 		)
-		(pin "IFH_H" input
+		(pin "IFH_P" input
 			(at 66.04 59.69 180)
 			(effects
