File: bms-main.kicad_pcb (KiCad board)
At the start: 4 copper layers, 49 x 49.9 mm, 69 parts, among them J1 CONN HEADER VERT 2POS 1.5MM, J2 CONN HEADER VERT 2POS 1.5MM, J3 CONN HEADER VERT 2POS 1.5MM, J4 CONN HEADER VERT 4POS 2.5MM, J5 PIN HEADER 2.54MM PITCH STR D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, J6 XT60PW-M, J7 XT60PW-M, U1 TLE9015DQUXUMA1, U2 STM32L433CCU6, U3 IC TRANSCEIVER 1/1 8SO, U4 INA181A3IDBVR, X1 CRYSTAL 32.0000MHZ 10PF SMD

Commit message: added logo
Parts:
- added G***: LOGO, footprints:electriumlogo15, F.Cu at (149.4, 52.8)
- added G***: LOGO, footprints:dog, B.Cu at (148.6, 59.0)
Other:
- board text added: "BMS Main"
- board text added: "Eleanor W"
